File: hardware/0.1/ecp5-mini.kicad_sch (KiCad schematic)
At the start: 22 parts, among them J3 S7 Mini, J4 S7 Mini, U1 ECP5U_12_CABGA256, X1 DSC6101CI2A-016

Commit message: half IO routed
Connections:
- net LED_0: now also U1.R13 (PR41C/+/RDQ44); no longer U1.T14 (PR41D/-/RDQ44)
- net LED_1: now also U1.T14 (PR41D/-/RDQ44); no longer U1.R14 (PR41B/-/HS/RDQ44)
- net LED_2: now also U1.R14 (PR41B/-/HS/RDQ44); no longer U1.T15 (PR38D/-/RDQ44)
- net LED_3: now also U1.P14 (PR38B/-/HS/RDQ44); no longer U1.R15 (PR38C/+/RDQ44)
- net LED_B: now also U1.T13 (PR44B/-/HS/RDQSN44); no longer U1.R13 (PR41C/+/RDQ44)
- net LED_G: now also U1.P13 (PR41A/+/HS/RDQ44); no longer U1.T13 (PR44B/-/HS/RDQSN44)
- net PORT_A0: now also U1.T15 (PR38D/-/RDQ44); no longer U1.P13 (PR41A/+/HS/RDQ44)
- net PORT_A1: now also U1.R16 (PR35B/-/VREF1_3/HS/RDQ32); no longer U1.P15 (PR32B/-/HS/RDQSN32)
- net PORT_A2: now also U1.P15 (PR32B/-/HS/RDQSN32); no longer U1.P14 (PR38B/-/HS/RDQ44)
- net PORT_A4: now also U1.R15 (PR38C/+/RDQ44); no longer U1.R16 (PR35B/-/VREF1_3/HS/RDQ32)
- net PORT_B0: now also U1.L15 (PR26B/-/PCLKC3_1/HS/RDQ32); no longer U1.L14 (PR32C/+/RDQ32)
- net PORT_B1: now also U1.K15 (PR23D/-/PCLKC2_0/RDQ20); no longer U1.L15 (PR26B/-/PCLKC3_1/HS/RDQ32)
- net PORT_B2: now also U1.J15 (PR23B/-/PCLKC2_1/HS/RDQ20); no longer U1.K15 (PR23D/-/PCLKC2_0/RDQ20)
- net PORT_B3: now also U1.K14 (PR20D/-/RDQ20); no longer U1.J15 (PR23B/-/PCLKC2_1/HS/RDQ20)
- net PORT_B7: now also U1.J14 (PR20C/+/GR_PCLK2_0/RDQ20); no longer U1.H15 (PR20B/-/HS/RDQSN20)
- net PORT_C0: now also U1.H15 (PR20B/-/HS/RDQSN20); no longer U1.G16 (PR20A/+/GR_PCLK2_1/HS/RDQS20)
- net PORT_C1: now also U1.G15 (PR14B/-/HS/RDQ20); no longer U1.F16 (PR14A/+/HS/RDQ20)
- net PORT_C2: now also U1.H14 (PR14D/-/RDQ20); no longer U1.E16 (PR11D/-/RDQ8)
- net PORT_C3: now also U1.E16 (PR11D/-/RDQ8); no longer U1.D16 (PR8A/+/HS/RDQS8)
- net PORT_C4: now also U1.G16 (PR20A/+/GR_PCLK2_1/HS/RDQS20); no longer U1.G15 (PR14B/-/HS/RDQ20)
- net PORT_C5: now also U1.F16 (PR14A/+/HS/RDQ20); no longer U1.F15 (PR11C/+/RDQ8)
- net PORT_C6: now also U1.G14 (PR14C/+/VREF1_2/RDQ20); no longer U1.E15 (PR8B/-/HS/RDQSN8)
- net PORT_C7: now also U1.F15 (PR11C/+/RDQ8); no longer U1.D14 (PR2D/-/RDQ8)
- net PORT_D0: now also U1.E15 (PR8B/-/HS/RDQSN8); no longer U1.C16 (PR5A/+/HS/RDQ8)
- net PORT_D1: now also U1.C15 (PR5B/-/HS/RDQ8); no longer U1.B16 (PR2A/+/HS/RDQ8)
- net PORT_D2: now also U1.D14 (PR2D/-/RDQ8); no longer U1.B15 (PR2B/-/S0_IN/HS/RDQ8)
- net PORT_D3: now also U1.B15 (PR2B/-/S0_IN/HS/RDQ8); no longer U1.C13 (PT60B/-)
- net PORT_D4: now also U1.D16 (PR8A/+/HS/RDQS8); no longer U1.C15 (PR5B/-/HS/RDQ8)
- net PORT_D5: now also U1.C16 (PR5A/+/HS/RDQ8); no longer U1.C14 (PR2C/+/RDQ8)
- net PORT_D6: now also U1.C14 (PR2C/+/RDQ8); no longer U1.D13 (PT62A/+)
- net PORT_D7: now also U1.B16 (PR2A/+/HS/RDQ8); no longer U1.D12 (PT58A/+)
- net USB_PU: now reaches U1.A8 (PT29B/-/PCLKC0_0)
- net SD_DAT0: now reaches U1.D10 (PT47A/+)
- net USB_D-: now reaches U1.D9 (PT40A/+)
- net SD_DAT1: now reaches U1.E10 (PT47B/-)
- net SD_DET: now reaches U1.E12 (PT58B/-)
- net SD_DAT2: now reaches U1.E13 (PT62B/-)
- net USB_D+: now reaches U1.E9 (PT40B/-)
- new net SD_CLK: U1.D12 (PT58A/+)
- new net SD_CMD: U1.D13 (PT62A/+)
- new net SD_DAT3: U1.C13 (PT60B/-)
Other:
- sheet LEDs ports: added none; removed LED_B, LED_G, LED_R
- note added: "LENGTH MATCHING: id: USB netnames: "/USB_D*" tolerance: 1.27 mm vialength: 1.6 mm"
- note added: "LENGTH MATCHING: id: hyperram netnames: "/HR_*" tolerance: 1.27 mm vialength: 1.6 mm"
- note removed: "LENGTH MATCHING: id: hyperram_dq_rwds netnames: "/HR_*" tolerance: 1.27 mm vialength: 1.6 mm"

Commit message: unrouted = 0
Connections:
- net FPGA_OK: now also U1.A6 (PT18B/-)
- net LED_USR: now also U1.A5 (PT18A/+)
- net PORT_E0: now also U1.C1 (PL5A/+/HS/LDQ8)
- net PORT_E1: now also U1.B1 (PL2A/+/HS/LDQ8)
- net PORT_E2: now also U1.A2 (PT4A/+)
- net PORT_E3: now also U1.A3 (PT6A/+)
- net PORT_E4: now also U1.C2 (PL5B/-/HS/LDQ8)
- net PORT_E5: now also U1.B2 (PL2B/-/HS/LDQ8)
- net PORT_E6: now also U1.B3 (PT4B/-)
- net PORT_E7: now also U1.A4 (PT6B/-)
- net PORT_F0: now also U1.K1 (PL23C/+/PCLKT7_0/LDQ20)
- net PORT_F1: now also U1.J1 (PL23A/+/PCLKT7_1/HS/LDQ20)
- net PORT_F2: now also U1.G1 (PL20A/+/GR_PCLK7_1/HS/LDQS20)
- net PORT_F3: now also U1.F1 (PL14A/+/HS/LDQ20)
- net PORT_F4: now also U1.K2 (PL23D/-/PCLKC7_0/LDQ20)
- net PORT_F5: now also U1.J2 (PL23B/-/PCLKC7_1/HS/LDQ20)
- net PORT_F6: now also U1.H2 (PL20B/-/HS/LDQSN20)
- net PORT_F7: now also U1.G2 (PL14B/-/HS/LDQ20)
- net PORT_G0: now also U1.N1 (PL32A/+/HS/LDQS32)
- net PORT_G1: now also U1.M1 (PL26C/+/PCLKT6_0/LDQ32)
- net PORT_G2: now also U1.L1 (PL26A/+/PCLKT6_1/HS/LDQ32)
- net PORT_G3: now also U1.L3 (PL32C/+/LDQ32)
- net PORT_G4: now also U1.P2 (PL32B/-/HS/LDQSN32)
- net PORT_G5: now also U1.M2 (PL26D/-/PCLKC6_0/LDQ32)
- net PORT_G6: now also U1.L2 (PL26B/-/PCLKC6_1/HS/LDQ32)
- net PORT_G7: now also U1.M3 (PL32D/-/LDQ32)
- net PORT_H0: now also U1.R2 (PL38C/+/LDQ44)
- net PORT_H1: now also U1.P4 (PL41A/+/HS/LDQ44)
- net PORT_H2: now also U1.N4 (PL38A/+/HS/LDQ44)
- net PORT_H3: now also U1.P1 (PL35A/+/HS/LDQ32)
- net PORT_H4: now also U1.T2 (PL38D/-/LDQ44)
- net PORT_H5: now also U1.R3 (PL41B/-/HS/LDQ44)
- net PORT_H6: now also U1.P3 (PL38B/-/HS/LDQ44)
- net PORT_H7: now also U1.R1 (PL35B/-/VREF1_6/HS/LDQ32)

Commit message: all DRC / ERC errors signed off
Connections:
- no-connect marks 0 -> 84
Other:
- moved on the sheet: C14, J3, J4, X1
