File: hardware/0.1/ecp5-mini.kicad_sch (KiCad schematic)
At the start: 28 parts, among them J3 S7 Mini, J4 S7 Mini, U1 ECP5U_12_CABGA256, X1 DSC6101CI2A-016

Commit message: quad pmod looks good
Parts:
- FID1, FID2, FID3, FID4, FID5, FID6: DNP (none) -> DNP
Changed lines of the file:
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@@
   (page 1 5)
   (paper "A3")
+  (bus_alias "LED" (members "LED_[0..7]" "LED_R" "LED_G" "LED_B"))
+  (bus_alias "HYPERRAM" (members "HR_nRST" "HR_nCS" "HR_CK_N" "HR_RWDS" "HR_DQ[0..7]" "HR_CK"))
+  (bus_alias "USB" (members "USB_D-" "USB_D+" "USB_PU"))
   (bus_alias "SD" (members "SD_DAT[0..3]" "SD_CMD" "SD_CLK" "SD_DET"))
-  (bus_alias "USB" (members "USB_D-" "USB_D+" "USB_PU"))
-  (bus_alias "HYPERRAM" (members "HR_nRST" "HR_nCS" "HR_CK_N" "HR_RWDS" "HR_DQ[0..7]" "HR_CK"))
-  (bus_alias "LED" (members "LED_[0..7]" "LED_R" "LED_G" "LED_B"))
   (junction (at 60.96 63.5) (diameter 1.016) (color 0 0 0 0))
   (junction (at 62.23 177.8) (diameter 1.016) (color 0 0 0 0))
@@
   (junction (at 358.14 196.85) (diameter 1.016) (color 0 0 0 0))
   (junction (at 358.14 198.12) (diameter 1.016) (color 0 0 0 0))
+  (no_connect (at 50.8 119.38))
+  (no_connect (at 208.28 224.79))
+  (no_connect (at 207.01 91.44))
+  (no_connect (at 50.8 241.3))
+  (no_connect (at 133.35 132.08))
+  (no_connect (at 50.8 99.06))
+  (no_connect (at 208.28 252.73))
+  (no_connect (at 133.35 137.16))
+  (no_connect (at 207.01 119.38))
+  (no_connect (at 207.01 99.06))
+  (no_connect (at 208.28 260.35))
+  (no_connect (at 208.28 227.33))
+  (no_connect (at 50.8 218.44))
+  (no_connect (at 130.81 269.24))
+  (no_connect (at 208.28 262.89))
+  (no_connect (at 133.35 99.06))
+  (no_connect (at 130.81 261.62))
+  (no_connect (at 130.81 266.7))
+  (no_connect (at 50.8 93.98))
+  (no_connect (at 207.01 93.98))
+  (no_connect (at 207.01 116.84))
+  (no_connect (at 130.81 271.78))
+  (no_connect (at 50.8 208.28))
+  (no_connect (at 133.35 134.62))
+  (no_connect (at 130.81 220.98))
+  (no_connect (at 50.8 236.22))
+  (no_connect (at 50.8 91.44))
+  (no_connect (at 208.28 229.87))
+  (no_connect (at 130.81 264.16))
+  (no_connect (at 50.8 231.14))
+  (no_connect (at 130.81 213.36))
+  (no_connect (at 50.8 238.76))
+  (no_connect (at 130.81 274.32))
+  (no_connect (at 133.35 114.3))
+  (no_connect (at 208.28 199.39))
+  (no_connect (at 208.28 242.57))
+  (no_connect (at 50.8 195.58))
+  (no_connect (at 50.8 220.98))
+  (no_connect (at 50.8 134.62))
+  (no_connect (at 208.28 232.41))
+  (no_connect (at 50.8 121.92))
+  (no_connect (at 207.01 96.52))
+  (no_connect (at 207.01 160.02))
+  (no_connect (at 208.28 240.03))
+  (no_connect (at 130.81 233.68))
+  (no_connect (at 207.01 157.48))
+  (no_connect (at 208.28 201.93))
+  (no_connect (at 133.35 111.76))
+  (no_connect (at 50.8 200.66))
+  (no_connect (at 208.28 222.25))
+  (no_connect (at 208.28 214.63))
+  (no_connect (at 130.81 210.82))
+  (no_connect (at 130.81 208.28))
+  (no_connect (at 133.35 109.22))
+  (no_connect (at 207.01 149.86))
+  (no_connect (at 50.8 104.14))
+  (no_connect (at 130.81 236.22))
+  (no_connect (at 130.81 231.14))
+  (no_connect (at 208.28 219.71))
+  (no_connect (at 207.01 152.4))
+  (no_connect (at 130.81 205.74))
+  (no_connect (at 208.28 245.11))
+  (no_connect (at 50.8 129.54))
+  (no_connect (at 207.01 147.32))
+  (no_connect (at 50.8 96.52))
+  (no_connect (at 133.35 96.52))
+  (no_connect (at 208.28 217.17))
+  (no_connect (at 50.8 106.68))
+  (no_connect (at 50.8 101.6))
+  (no_connect (at 208.28 250.19))
+  (no_connect (at 130.81 223.52))
+  (no_connect (at 208.28 247.65))
+  (no_connect (at 133.35 106.68))
+  (no_connect (at 133.35 139.7))
   (no_connect (at 50.8 132.08))
-  (no_connect (at 133.35 96.52))
-  (no_connect (at 50.8 121.92))
-  (no_connect (at 50.8 99.06))
-  (no_connect (at 208.28 222.25))
-  (no_connect (at 133.35 99.06))
-  (no_connect (at 207.01 116.84))
-  (no_connect (at 208.28 247.65))
-  (no_connect (at 133.35 134.62))
-  (no_connect (at 50.8 93.98))
+  (no_connect (at 208.28 209.55))
+  (no_connect (at 50.8 139.7))
+  (no_connect (at 50.8 198.12))
   (no_connect (at 50.8 127))
-  (no_connect (at 50.8 134.62))
-  (no_connect (at 50.8 218.44))
+  (no_connect (at 50.8 109.22))
+  (no_connect (at 50.8 243.84))
   (no_connect (at 207.01 154.94))
-  (no_connect (at 207.01 96.52))
-  (no_connect (at 50.8 231.14))
-  (no_connect (at 208.28 199.39))
-  (no_connect (at 207.01 119.38))
-  (no_connect (at 208.28 224.79))
-  (no_connect (at 50.8 139.7))
-  (no_connect (at 50.8 238.76))
-  (no_connect (at 50.8 96.52))
-  (no_connect (at 207.01 152.4))
   (no_connect (at 208.28 212.09))
-  (no_connect (at 208.28 232.41))
-  (no_connect (at 208.28 250.19))
-  (no_connect (at 130.81 208.28))
-  (no_connect (at 130.81 269.24))
-  (no_connect (at 50.8 200.66))
-  (no_connect (at 208.28 245.11))
-  (no_connect (at 130.81 236.22))
-  (no_connect (at 133.35 111.76))
-  (no_connect (at 208.28 214.63))
-  (no_connect (at 50.8 129.54))
-  (no_connect (at 207.01 149.86))
-  (no_connect (at 130.81 210.82))
-  (no_connect (at 130.81 233.68))
-  (no_connect (at 50.8 243.84))
-  (no_connect (at 50.8 236.22))
-  (no_connect (at 208.28 252.73))
-  (no_connect (at 208.28 209.55))
-  (no_connect (at 133.35 114.3))
-  (no_connect (at 133.35 132.08))
-  (no_connect (at 207.01 157.48))
-  (no_connect (at 130.81 264.16))
-  (no_connect (at 50.8 198.12))
-  (no_connect (at 207.01 93.98))
-  (no_connect (at 50.8 106.68))
-  (no_connect (at 130.81 223.52))
-  (no_connect (at 130.81 205.74))
-  (no_connect (at 207.01 99.06))
-  (no_connect (at 130.81 266.7))
-  (no_connect (at 208.28 227.33))
-  (no_connect (at 208.28 229.87))
-  (no_connect (at 50.8 208.28))
-  (no_connect (at 133.35 137.16))
-  (no_connect (at 207.01 160.02))
-  (no_connect (at 130.81 220.98))
-  (no_connect (at 208.28 219.71))
-  (no_connect (at 130.81 271.78))
-  (no_connect (at 130.81 261.62))
-  (no_connect (at 50.8 220.98))
-  (no_connect (at 130.81 274.32))
-  (no_connect (at 50.8 119.38))
-  (no_connect (at 208.28 217.17))
-  (no_connect (at 130.81 213.36))
-  (no_connect (at 133.35 139.7))
-  (no_connect (at 208.28 201.93))
-  (no_connect (at 208.28 260.35))
-  (no_connect (at 50.8 91.44))
-  (no_connect (at 133.35 106.68))
-  (no_connect (at 50.8 101.6))
-  (no_connect (at 207.01 91.44))
-  (no_connect (at 208.28 242.57))
-  (no_connect (at 130.81 231.14))
-  (no_connect (at 50.8 104.14))
-  (no_connect (at 208.28 240.03))
-  (no_connect (at 207.01 147.32))
-  (no_connect (at 50.8 109.22))
-  (no_connect (at 50.8 195.58))
-  (no_connect (at 50.8 241.3))
-  (no_connect (at 133.35 109.22))
-  (no_connect (at 208.28 262.89))
   (no_connect (at 50.8 116.84))
   (bus_entry (at 62.23 203.2) (size 2.54 -2.54)
@@
       (effects (font (size 1.27 1.27)) hide)
     )
+    (property "DNP" "DNP" (id 4) (at 358.14 240.03 0)
+      (effects (font (size 1.27 1.27)) hide)
+    )
   )
   (symbol (lib_id "Mechanical:Fiducial") (at 358.14 243.84 0) (unit 1)
@@
       (effects (font (size 1.27 1.27)) hide)
     )
+    (property "DNP" "DNP" (id 4) (at 358.14 243.84 0)
+      (effects (font (size 1.27 1.27)) hide)
+    )
   )
   (symbol (lib_id "Mechanical:Fiducial") (at 358.14 247.65 0) (unit 1)
@@
       (effects (font (size 1.27 1.27)) hide)
     )
+    (property "DNP" "DNP" (id 4) (at 358.14 247.65 0)
+      (effects (font (size 1.27 1.27)) hide)
+    )
   )
   (symbol (lib_id "Mechanical:Fiducial") (at 370.84 240.03 0) (unit 1)
@@
       (effects (font (size 1.27 1.27)) hide)
     )
+    (property "DNP" "DNP" (id 4) (at 370.84 240.03 0)
+      (effects (font (size 1.27 1.27)) hide)
+    )
   )
   (symbol (lib_id "Mechanical:Fiducial") (at 370.84 243.84 0) (unit 1)
@@
       (effects (font (size 1.27 1.27)) hide)
     )
+    (property "DNP" "DNP" (id 4) (at 370.84 243.84 0)
+      (effects (font (size 1.27 1.27)) hide)
+    )
   )
   (symbol (lib_id "Mechanical:Fiducial") (at 370.84 247.65 0) (unit 1)
@@
       (effects (font (size 1.27 1.27)) hide)
     )
+    (property "DNP" "DNP" (id 4) (at 370.84 247.65 0)
+      (effects (font (size 1.27 1.27)) hide)
+    )

Commit message: update readme following r0.1 bringup
Parts:
- R22, R23, R5: value 2K2 -> 1K5; LCSC C25933 -> C25867; MPN 0402WGJ0222TCE -> 0402WGF1501TCE
Changed lines of the file:
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@@
   (junction (at 358.14 196.85) (diameter 1.016) (color 0 0 0 0))
   (junction (at 358.14 198.12) (diameter 1.016) (color 0 0 0 0))
-  (no_connect (at 50.8 119.38))
-  (no_connect (at 208.28 224.79))
+  (no_connect (at 207.01 160.02))
+  (no_connect (at 208.28 222.25))
+  (no_connect (at 130.81 213.36))
   (no_connect (at 207.01 91.44))
-  (no_connect (at 50.8 241.3))
-  (no_connect (at 133.35 132.08))
-  (no_connect (at 50.8 99.06))
-  (no_connect (at 208.28 252.73))
-  (no_connect (at 133.35 137.16))
-  (no_connect (at 207.01 119.38))
   (no_connect (at 207.01 99.06))
-  (no_connect (at 208.28 260.35))
-  (no_connect (at 208.28 227.33))
-  (no_connect (at 50.8 218.44))
-  (no_connect (at 130.81 269.24))
-  (no_connect (at 208.28 262.89))
-  (no_connect (at 133.35 99.06))
-  (no_connect (at 130.81 261.62))
-  (no_connect (at 130.81 266.7))
-  (no_connect (at 50.8 93.98))
-  (no_connect (at 207.01 93.98))
   (no_connect (at 207.01 116.84))
-  (no_connect (at 130.81 271.78))
-  (no_connect (at 50.8 208.28))
-  (no_connect (at 133.35 134.62))
-  (no_connect (at 130.81 220.98))
-  (no_connect (at 50.8 236.22))
-  (no_connect (at 50.8 91.44))
-  (no_connect (at 208.28 229.87))
-  (no_connect (at 130.81 264.16))
-  (no_connect (at 50.8 231.14))
-  (no_connect (at 130.81 213.36))
-  (no_connect (at 50.8 238.76))
   (no_connect (at 130.81 274.32))
-  (no_connect (at 133.35 114.3))
+  (no_connect (at 50.8 91.44))
+  (no_connect (at 50.8 236.22))
   (no_connect (at 208.28 199.39))
-  (no_connect (at 208.28 242.57))
-  (no_connect (at 50.8 195.58))
-  (no_connect (at 50.8 220.98))
-  (no_connect (at 50.8 134.62))
-  (no_connect (at 208.28 232.41))
-  (no_connect (at 50.8 121.92))
   (no_connect (at 207.01 96.52))
-  (no_connect (at 207.01 160.02))
+  (no_connect (at 130.81 236.22))
+  (no_connect (at 50.8 134.62))
+  (no_connect (at 133.35 139.7))
+  (no_connect (at 50.8 243.84))
+  (no_connect (at 208.28 229.87))
   (no_connect (at 208.28 240.03))
-  (no_connect (at 130.81 233.68))
-  (no_connect (at 207.01 157.48))
-  (no_connect (at 208.28 201.93))
-  (no_connect (at 133.35 111.76))
-  (no_connect (at 50.8 200.66))
-  (no_connect (at 208.28 222.25))
-  (no_connect (at 208.28 214.63))
-  (no_connect (at 130.81 210.82))
-  (no_connect (at 130.81 208.28))
-  (no_connect (at 133.35 109.22))
+  (no_connect (at 207.01 147.32))
+  (no_connect (at 50.8 241.3))
+  (no_connect (at 133.35 99.06))
+  (no_connect (at 208.28 232.41))
   (no_connect (at 207.01 149.86))
+  (no_connect (at 130.81 264.16))
+  (no_connect (at 130.81 261.62))
+  (no_connect (at 208.28 262.89))
+  (no_connect (at 208.28 219.71))
+  (no_connect (at 133.35 137.16))
+  (no_connect (at 207.01 93.98))
+  (no_connect (at 130.81 223.52))
+  (no_connect (at 133.35 134.62))
+  (no_connect (at 50.8 101.6))
+  (no_connect (at 133.35 109.22))
+  (no_connect (at 133.35 111.76))
   (no_connect (at 50.8 104.14))
-  (no_connect (at 130.81 236.22))
+  (no_connect (at 50.8 121.92))
+  (no_connect (at 130.81 220.98))
   (no_connect (at 130.81 231.14))
-  (no_connect (at 208.28 219.71))
-  (no_connect (at 207.01 152.4))
+  (no_connect (at 50.8 119.38))
+  (no_connect (at 208.28 212.09))
+  (no_connect (at 50.8 220.98))
+  (no_connect (at 130.81 208.28))
   (no_connect (at 130.81 205.74))
-  (no_connect (at 208.28 245.11))
-  (no_connect (at 50.8 129.54))
-  (no_connect (at 207.01 147.32))
+  (no_connect (at 50.8 93.98))
+  (no_connect (at 208.28 227.33))
+  (no_connect (at 50.8 208.28))
+  (no_connect (at 50.8 231.14))
+  (no_connect (at 133.35 114.3))
   (no_connect (at 50.8 96.52))
-  (no_connect (at 133.35 96.52))
-  (no_connect (at 208.28 217.17))
-  (no_connect (at 50.8 106.68))
-  (no_connect (at 50.8 101.6))
-  (no_connect (at 208.28 250.19))
-  (no_connect (at 130.81 223.52))
-  (no_connect (at 208.28 247.65))
-  (no_connect (at 133.35 106.68))
-  (no_connect (at 133.35 139.7))
   (no_connect (at 50.8 132.08))
-  (no_connect (at 208.28 209.55))
+  (no_connect (at 208.28 201.93))
+  (no_connect (at 50.8 99.06))
+  (no_connect (at 133.35 106.68))
+  (no_connect (at 50.8 200.66))
+  (no_connect (at 130.81 271.78))
+  (no_connect (at 208.28 260.35))
+  (no_connect (at 130.81 269.24))
   (no_connect (at 50.8 139.7))
+  (no_connect (at 130.81 266.7))
+  (no_connect (at 50.8 109.22))
+  (no_connect (at 50.8 129.54))
+  (no_connect (at 208.28 224.79))
+  (no_connect (at 50.8 116.84))
+  (no_connect (at 50.8 106.68))
+  (no_connect (at 208.28 214.63))
+  (no_connect (at 130.81 210.82))
+  (no_connect (at 50.8 218.44))
+  (no_connect (at 207.01 119.38))
+  (no_connect (at 208.28 247.65))
+  (no_connect (at 208.28 245.11))
+  (no_connect (at 50.8 195.58))
+  (no_connect (at 50.8 238.76))
+  (no_connect (at 208.28 252.73))
+  (no_connect (at 208.28 242.57))
   (no_connect (at 50.8 198.12))
   (no_connect (at 50.8 127))
-  (no_connect (at 50.8 109.22))
-  (no_connect (at 50.8 243.84))
+  (no_connect (at 208.28 250.19))
+  (no_connect (at 208.28 217.17))
+  (no_connect (at 130.81 233.68))
+  (no_connect (at 207.01 152.4))
+  (no_connect (at 133.35 132.08))
+  (no_connect (at 208.28 209.55))
   (no_connect (at 207.01 154.94))
-  (no_connect (at 208.28 212.09))
-  (no_connect (at 50.8 116.84))
+  (no_connect (at 207.01 157.48))
+  (no_connect (at 133.35 96.52))
   (bus_entry (at 62.23 203.2) (size 2.54 -2.54)
     (stroke (width 0.1524) (type solid) (color 0 0 0 0))
@@
       (effects (font (size 1.27 1.27)) (justify left))
     )
-    (property "Value" "2K2" (id 1) (at 377.825 197.485 0)
+    (property "Value" "1K5" (id 1) (at 377.825 197.485 0)
       (effects (font (size 1.27 1.27)) (justify left))
     )
@@
       (effects (font (size 1.27 1.27)) hide)
     )
-    (property "LCSC" "C25933" (id 4) (at 375.285 196.215 0)
+    (property "LCSC" "C25867" (id 4) (at 375.285 196.215 0)
       (effects (font (size 1.27 1.27)) hide)
     )
-    (property "MPN" "0402WGJ0222TCE" (id 5) (at 375.285 196.215 0)
+    (property "MPN" "0402WGF1501TCE" (id 5) (at 375.285 196.215 0)
       (effects (font (size 1.27 1.27)) hide)
     )
@@
       (effects (font (size 1.27 1.27)) (justify left))
     )
-    (property "Value" "2K2" (id 1) (at 389.255 197.485 0)
+    (property "Value" "1K5" (id 1) (at 389.255 197.485 0)
       (effects (font (size 1.27 1.27)) (justify left))
     )
@@
       (effects (font (size 1.27 1.27)) hide)
     )
-    (property "LCSC" "C25933" (id 4) (at 386.715 196.215 0)
+    (property "LCSC" "C25867" (id 4) (at 386.715 196.215 0)
       (effects (font (size 1.27 1.27)) hide)
     )
-    (property "MPN" "0402WGJ0222TCE" (id 5) (at 386.715 196.215 0)
+    (property "MPN" "0402WGF1501TCE" (id 5) (at 386.715 196.215 0)
       (effects (font (size 1.27 1.27)) hide)
     )
@@
       (effects (font (size 1.27 1.27)) (justify left))
     )
-    (property "Value" "2K2" (id 1) (at 400.685 197.485 0)
+    (property "Value" "1K5" (id 1) (at 400.685 197.485 0)
       (effects (font (size 1.27 1.27)) (justify left))
     )
@@
       (effects (font (size 1.27 1.27)) hide)
     )
-    (property "LCSC" "C25933" (id 4) (at 398.145 196.215 0)
+    (property "LCSC" "C25867" (id 4) (at 398.145 196.215 0)
       (effects (font (size 1.27 1.27)) hide)
     )
-    (property "MPN" "0402WGJ0222TCE" (id 5) (at 398.145 196.215 0)
+    (property "MPN" "0402WGF1501TCE" (id 5) (at 398.145 196.215 0)
       (effects (font (size 1.27 1.27)) hide)
     )
@@
     )
     (path "/7ad9e016-ef6c-4e7d-bf98-b182394deaaa"
-      (reference "R5") (unit 1) (value "2K2") (footprint "Resistor_SMD:R_0402_1005Metric")
+      (reference "R5") (unit 1) (value "1K5") (footprint "Resistor_SMD:R_0402_1005Metric")
     )
     (path "/eb9d8bd1-e24f-46ce-9823-243f60c5e0fe"
-      (reference "R22") (unit 1) (value "2K2") (footprint "Resistor_SMD:R_0402_1005Metric")
+      (reference "R22") (unit 1) (value "1K5") (footprint "Resistor_SMD:R_0402_1005Metric")
     )
     (path "/7653e333-6391-493a-8f32-a3e0174495ff"
-      (reference "R23") (unit 1) (value "2K2") (footprint "Resistor_SMD:R_0402_1005Metric")
+      (reference "R23") (unit 1) (value "1K5") (footprint "Resistor_SMD:R_0402_1005Metric")
     )
     (path "/044da9c4-4a64-4ef9-9440-36766290b369"
@@
     )
     (path "/dc977d07-e2f1-4e46-a04d-d09b8b7fb491/882e829a-4dce-4846-8590-2c97e75344ea"
-      (reference "R21") (unit 1) (value "2K2") (footprint "Resistor_SMD:R_0402_1005Metric")
+      (reference "R21") (unit 1) (value "1K5") (footprint "Resistor_SMD:R_0402_1005Metric")
     )
     (path "/dc977d07-e2f1-4e46-a04d-d09b8b7fb491/daf7bb8c-3299-4f8b-9706-f5fe189e6057"

Commit message: update BOM
Parts:
- D1, D12, D3: Notes (none) -> If not using exact PN, may want to increase resistor values
- FID1, FID2, FID3, FID4, FID5, FID6, J3, J4, LOGO1, LOGO2: now left out of the parts list
- U1: Manufacturer Lattice -> Lattice Semiconductor
