File: hardware/0.1/power.kicad_sch (KiCad schematic)
At the start: 28 parts, among them U1 ECP5U_12_CABGA256, U2 TLV73325PDBV, U3 TLV62568DBV, U5 TLV62568DBV

Commit message: add part numbers
Parts:
- C1, C2: LCSC (none) -> C19666; MPN (none) -> CL10A475KO8NNNC; Manufacturer (none) -> Samsung Electro-Mechanics
- C10, C7: LCSC C100082 -> C86295; MPN CL10B225KP8NNNC -> CL10A226MP8NUNE; Manufacturer (none) -> Samsung Electro-Mechanics
- C21, C22: LCSC (none) -> C368809; MPN (none) -> CL05A475KP5NRNC; Manufacturer (none) -> Samsung Electro-Mechanics
- C3, C4: LCSC (none) -> C5673; MPN (none) -> CL10A105KA8NNNC; Manufacturer (none) -> Samsung Electro-Mechanics
- C37, C38, C39, C40, C41, C42, C43: LCSC (none) -> C1525; MPN (none) -> CL05B104KO5NNNC; Manufacturer (none) -> Samsung Electro-Mechanics
- C5: LCSC (none) -> C92487; MPN (none) -> CL10A106MO8NQNC; Manufacturer (none) -> Samsung Electro-Mechanics
- C8, C9: LCSC (none) -> C86292; MPN (none) -> CL05C6R8DB5NNNC; Manufacturer (none) -> Samsung Electro-Mechanics
- L1, L2: Manufacturer (none) -> Sunltech Tech
- R1: LCSC (none) -> C58827; Manufacturer (none) -> UNI-ROYAL(Uniroyal Elec)
- R2: LCSC (none) -> C25792; MPN RC0402FR-0747KL -> 0402WGF4702TCE; Manufacturer (none) -> UNI-ROYAL(Uniroyal Elec)
- R3: LCSC (none) -> C26988; Manufacturer (none) -> UNI-ROYAL(Uniroyal Elec)
- R4: LCSC (none) -> C25741; Manufacturer (none) -> UNI-ROYAL(Uniroyal Elec)
- U1: MPN (none) -> LFE5U-12F-8BG256C; Manufacturer (none) -> Lattice; Mouser (none) -> 842-LFE5U12F8BG256C
- U2: MPN (none) -> TLV73325PDBVR; Manufacturer (none) -> Texas Instruments; Mouser (none) -> 595-TLV73325PDBVR
- U3, U5: Manufacturer (none) -> Texas Instruments

Commit message: design review done
Parts:
- U1: MPN LFE5U-12F-8BG256C -> LFE5U12F8BG256C
Changed lines of the file:
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@@
     )
   )
-  (symbol (lib_id "Device:L") (at 58.42 39.37 90) (unit 1)
+  (symbol (lib_name "Device:L_1") (lib_id "Device:L") (at 58.42 39.37 90) (unit 1)
     (in_bom yes) (on_board yes)
     (property "Reference" "L1" (id 0) (at 58.42 34.29 90))
@@
       (effects (font (size 1.524 1.524)) (justify right) hide)
     )
-    (property "MPN" "LFE5U-12F-8BG256C" (id 4) (at 215.9 48.26 0)
-      (effects (font (size 1.27 1.27)) hide)
-    )
     (property "Manufacturer" "Lattice" (id 5) (at 215.9 48.26 0)
       (effects (font (size 1.27 1.27)) hide)
@@
       (effects (font (size 1.27 1.27)) hide)
     )
+    (property "MPN" "LFE5U12F8BG256C" (id 4) (at 215.9 48.26 0)
+      (effects (font (size 1.27 1.27)) hide)
+    )

Commit message: update readme following r0.1 bringup
Parts:
- C10, C7: LCSC C86295 -> (none); MPN CL10A226MP8NUNE -> (none)
Changed lines of the file:
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@@
       (effects (font (size 1.27 1.27)) hide)
     )
-    (property "LCSC" "C86295" (id 4) (at 63.5 82.55 0)
+    (property "LCSC" "" (id 4) (at 63.5 82.55 0)
       (effects (font (size 1.27 1.27)) hide)
     )
-    (property "MPN" "CL10A226MP8NUNE" (id 5) (at 63.5 82.55 0)
+    (property "MPN" "" (id 5) (at 63.5 82.55 0)
       (effects (font (size 1.27 1.27)) hide)
     )
@@
       (effects (font (size 1.27 1.27)) hide)
     )
-    (property "LCSC" "C86295" (id 4) (at 72.39 82.55 0)
+    (property "LCSC" "" (id 4) (at 72.39 82.55 0)
       (effects (font (size 1.27 1.27)) hide)
     )
-    (property "MPN" "CL10A226MP8NUNE" (id 5) (at 72.39 82.55 0)
+    (property "MPN" "" (id 5) (at 72.39 82.55 0)
       (effects (font (size 1.27 1.27)) hide)
     )

Commit message: update BOM
Parts:
- C10, C7: value 22u -> 10u; LCSC (none) -> C92487; MPN (none) -> CL10A106MO8NQNC
- L1, L2: Mouser (none) -> 81-LQM21PN2R2NGCDCD; Notes (none) -> Mouser Murata, LCSC compatiable
- U1: Manufacturer Lattice -> Lattice Semiconductor
- U2: LCSC (none) -> C882825
- U3, U5: Mouser (none) -> 595-TLV62568DBVR
Other:
- note added: "V_{out} = 0.6V * (1 + R1/R2) 1v11 = 0.6 * (1 + 84k5/100k) 1v1 @ 1A"
- note added: "V_{out} = 0.6V * (1 + R1/R2) 3v28 = 0.6 * (1 + 210k/47k) 3v3 @ 1A"
- note removed: "V_{out} = 0.6V * (1 - R1 / R2) 1v11 = 0.6 * (1 - 84k5/ 100k) 1v1 @ 1A"
- note removed: "V_{out} = 0.6V * (1 - R1 / R2) 3v28 = 0.6 * (1 - 210k/ 47k) 3v3 @ 1A"
Changed lines of the file:
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@@
-(kicad_sch (version 20200828) (generator eeschema)
-  (page 5 5)
+(kicad_sch (version 20201015) (generator eeschema)
+  (page 1 5)
   (paper "A4")
   (junction (at 26.67 43.18) (diameter 1.016) (color 0 0 0 0))
@@
     (effects (font (size 5 5)) (justify right bottom))
   )
-  (text "V_{out} = 0.6V * (1 - R1 / R2)\n3v28 = 0.6 * (1 - 210k/ 47k)\n3v3 @ 1A"
+  (text "V_{out} = 0.6V * (1 + R1/R2)\n3v28 = 0.6 * (1 + 210k/47k)\n3v3 @ 1A"
     (at 93.98 47.371 0)
     (effects (font (size 1.27 1.27)) (justify left bottom))
   )
-  (text "V_{out} = 0.6V * (1 - R1 / R2)\n1v11 = 0.6 * (1 - 84k5/ 100k)\n1v1 @ 1A"
+  (text "V_{out} = 0.6V * (1 + R1/R2)\n1v11 = 0.6 * (1 + 84k5/100k)\n1v1 @ 1A"
     (at 104.14 90.17 0)
     (effects (font (size 1.27 1.27)) (justify left bottom))
@@
       (effects (font (size 1.27 1.27)) hide)
     )
+    (property "Mouser" "81-LQM21PN2R2NGCDCD " (id 4) (at 58.42 39.37 0)
+      (effects (font (size 1.27 1.27)) hide)
+    )
+    (property "Notes" "Mouser Murata, LCSC compatiable" (id 5) (at 58.42 39.37 0)
+      (effects (font (size 1.27 1.27)) hide)
+    )
   )
   (symbol (lib_id "Device:L") (at 58.42 77.47 90) (unit 1)
@@
       (effects (font (size 1.27 1.27)) hide)
     )
+    (property "Mouser" "81-LQM21PN2R2NGCDCD " (id 4) (at 58.42 77.47 0)
+      (effects (font (size 1.27 1.27)) hide)
+    )
+    (property "Notes" "Mouser Murata, LCSC compatiable" (id 5) (at 58.42 77.47 0)
+      (effects (font (size 1.27 1.27)) hide)
+    )
   )
   (symbol (lib_id "power:GND") (at 26.67 54.61 0) (unit 1)
@@
       (effects (font (size 1.27 1.27)) (justify left))
     )
-    (property "Value" "22u" (id 1) (at 66.04 83.82 0)
+    (property "Value" "10u" (id 1) (at 66.04 83.82 0)
       (effects (font (size 1.27 1.27)) (justify left))
     )
@@
       (effects (font (size 1.27 1.27)) hide)
     )
-    (property "LCSC" "" (id 4) (at 63.5 82.55 0)
-      (effects (font (size 1.27 1.27)) hide)
-    )
-    (property "MPN" "" (id 5) (at 63.5 82.55 0)
+    (property "LCSC" "C92487" (id 4) (at 63.5 82.55 0)
+      (effects (font (size 1.27 1.27)) hide)
+    )
+    (property "MPN" "CL10A106MO8NQNC" (id 5) (at 63.5 82.55 0)
       (effects (font (size 1.27 1.27)) hide)
     )
@@
       (effects (font (size 1.27 1.27)) (justify left))
     )
-    (property "Value" "22u" (id 1) (at 74.93 83.82 0)
+    (property "Value" "10u" (id 1) (at 74.93 83.82 0)
       (effects (font (size 1.27 1.27)) (justify left))
     )
@@
       (effects (font (size 1.27 1.27)) hide)
     )
-    (property "LCSC" "" (id 4) (at 72.39 82.55 0)
-      (effects (font (size 1.27 1.27)) hide)
-    )
-    (property "MPN" "" (id 5) (at 72.39 82.55 0)
+    (property "LCSC" "C92487" (id 4) (at 72.39 82.55 0)
+      (effects (font (size 1.27 1.27)) hide)
+    )
+    (property "MPN" "CL10A106MO8NQNC" (id 5) (at 72.39 82.55 0)
       (effects (font (size 1.27 1.27)) hide)
     )
@@
       (effects (font (size 1.27 1.27)) hide)
     )
+    (property "LCSC" "C882825" (id 4) (at 40.64 123.19 0)
+      (effects (font (size 1.27 1.27)) hide)
+    )
   )
   (symbol (lib_id "Regulator_Switching:TLV62568DBV") (at 44.45 45.72 0) (unit 1)
@@
       (effects (font (size 1.27 1.27)) hide)
     )
+    (property "Mouser" "595-TLV62568DBVR" (id 4) (at 44.45 45.72 0)
+      (effects (font (size 1.27 1.27)) hide)
+    )
   )
   (symbol (lib_id "Regulator_Switching:TLV62568DBV") (at 44.45 83.82 0) (unit 1)
@@
       (effects (font (size 1.27 1.27)) hide)
     )
+    (property "Mouser" "595-TLV62568DBVR" (id 4) (at 44.45 83.82 0)
+      (effects (font (size 1.27 1.27)) hide)
+    )
   )
   (symbol (lib_id "josh-ic:ECP5U_12_CABGA256") (at 215.9 48.26 0) (unit 1)
@@
       (effects (font (size 1.524 1.524)) (justify right) hide)
     )
-    (property "Manufacturer" "Lattice" (id 5) (at 215.9 48.26 0)
-      (effects (font (size 1.27 1.27)) hide)
-    )
+    (property "Manufacturer" "Lattice Semiconductor" (id 5) (at 215.9 48.26 0)
+      (effects (font (size 1.27 1.27)) hide)
+    )
