File: hardware/clock-test/clock-test.kicad_sch (KiCad schematic)
At the start: 78 parts, among them J3 S7 Mini, J4 S7 Mini

Commit message: clock-test laid out
Parts:
- added J1: PWR, Connector_PinHeader_2.54mm:PinHeader_1x02_P2.54mm_Vertical, symbol Connector:Conn_01x02_Male
- added Q1, Q2, Q3: DMG2302U, Package_TO_SOT_SMD:SOT-23, symbol Transistor_FET:DMG2302U
- added RN16: 10K, Resistor_SMD:R_Array_Convex_4x0603, symbol josh-passive:RN
- added SW1: SW_Push, josh-buttons-switches:Switch_SMT_SKPMAPE010, symbol Switch:SW_Push
Connections:
- net +3V3: now also RN16.4
- net +5V: now also J1.1 (Pin_1)
- net CAT_B: now also Q3.3 (D)
- net CAT_G: now also Q2.3 (D)
- net CAT_R: now also Q1.3 (D)
- net GND: now also J1.2 (Pin_2), Q1.2 (S), Q2.2 (S), Q3.2 (S), RN16.1, RN16.2, RN16.3, SW1.2
- net PORT_A0: now also RN3.8
- net PORT_A1: now also RN3.6
- net PORT_A2: now also RN2.8
- net PORT_A3: now also RN2.6
- net PORT_A4: now also RN3.7
- net PORT_A5: now also RN3.5
- net PORT_A6: now also RN2.7
- net PORT_A7: now also RN2.5
- net PORT_B0: now also RN1.8
- net PORT_B1: now also RN1.6
- net PORT_B2: now also RN15.8
- net PORT_B3: now also RN15.6
- net PORT_B4: now also RN1.7
- net PORT_B5: now also RN1.5
- net PORT_B6: now also RN15.7
- net PORT_B7: now also RN15.5
- net PORT_C0: now also RN14.8
- net PORT_C1: now also RN14.6
- net PORT_C2: now also RN13.8
- net PORT_C3: now also RN13.6
- net PORT_C4: now also RN14.7
- net PORT_C5: now also RN14.5
- net PORT_C6: now also RN13.7
- net PORT_C7: now also RN13.5
- net PORT_D0: now also RN11.5
- net PORT_D1: now also RN11.7
- net PORT_D2: now also RN12.5
- net PORT_D3: now also RN12.7
- net PORT_D4: now also RN11.6
- net PORT_D5: now also RN11.8
- net PORT_D6: now also RN12.6
- net PORT_D7: now also RN12.8
- net PORT_E0: now also RN9.5
- net PORT_E1: now also RN9.7
- net PORT_E2: now also RN10.5
- net PORT_E3: now also RN10.7
- net PORT_E4: now also RN9.6
- net PORT_E5: now also RN9.8
- net PORT_E6: now also RN10.6
- net PORT_E7: now also RN10.8
- net PORT_F0: now also RN7.5
- net PORT_F1: now also RN7.7
- net PORT_F2: now also RN8.5
- net PORT_F3: now also RN8.7
- net PORT_F4: now also RN7.6
- net PORT_F5: now also RN7.8
- net PORT_F6: now also RN8.6
- net PORT_F7: now also RN8.8
- net PORT_G0: now also RN5.5
- net PORT_G1: now also RN5.7
- net PORT_G2: now also RN6.5
- net PORT_G3: now also RN6.7
- net PORT_G4: now also RN5.6
- net PORT_G5: now also RN5.8
- net PORT_G6: now also RN6.6
- net PORT_G7: now also RN6.8
- net PORT_H0: now also RN4.8
- net PORT_H1: now also RN4.6
- net PORT_H2: now also Q3.1 (G), RN16.8
- net PORT_H3: now also Q1.1 (G), RN16.6
- net PORT_H4: now also RN4.7
- net PORT_H5: now also RN4.5
- net PORT_H6: now also Q2.1 (G), RN16.7
- net PORT_H7: now also RN16.5, SW1.1
