File: hardware/octa-pmod/octa-pmod.kicad_pcb (KiCad board)
At the start: 2 copper layers, 54.5 x 46.4 mm, 19 parts, among them J1 PMOD, J10 PMOD, J12 PWR, J14 PWR, J15 PMOD, J16 PMOD, J2 PMOD, J3 S7 Mini, J4 S7 Mini, J5 PWR, J6 PWR, J7 PMOD, J8 PMOD, J9 PMOD, M1 M3, M2 M3, M3 M3, M4 M3

Commit message: update readme following r0.1 bringup
Other:
- board text added: "JLCJLCJLCJLC"
Changed lines of the file:
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@@
+    (effects (font (size 1 1) (thickness 0.15)) (justify mirror))
+  )
+  (gr_text "JLCJLCJLCJLC" (at 115.7475 91.7 270) (layer "B.SilkS")
     (effects (font (size 1 1) (thickness 0.15)) (justify mirror))
   )
