File: hardware/octa-pmod-horizontal/octa-pmod.kicad_pcb (KiCad board)
At the start: 2 copper layers, 89 x 63.8 mm, 21 parts, among them J1 PMOD, J10 PMOD, J11 PWR, J12 PWR, J13 PWR, J14 PWR, J15 PMOD, J16 PMOD, J2 PMOD, J3 S7 Mini, J4 S7 Mini, J5 PWR, J6 PWR, J7 PMOD, J8 PMOD, J9 PMOD, M1 M3, M2 M3, M3 M3, M4 M3

Commit message: clean up routing
Routing:
- net /PORT_A7: track 16.2 -> 17.2 mm
- net /PORT_D2: track 23.1 -> 23.7 mm
- net /PORT_D1: track 23.1 -> 23.6 mm
- net /PORT_D0: track 23.1 -> 23.6 mm
Other:
- board text added: "BELOW PMODs PINOUT FLIPPED {0:3} = {4:7}"
- board text added: "NOTE: BELOW PMODs PINOUT FLIPPED {0:3} = {4:7}"
- board text removed: "BELOW PMODs PINOUT FLIPPED {0:3 = 4:7}"
- board text removed: "NOTE: BELOW PMODs PINOUT FLIPPED {0:3 = 4:7}"

Commit message: update readme following r0.1 bringup
Other:
- board text added: "JLCJLCJLCJLC"
Changed lines of the file:
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@@
   (gr_line (start 184 123.6) (end 101 123.6) (layer "Edge.Cuts") (width 0.1))
   (gr_arc (start 184 62.8) (end 187 62.8) (angle -90) (layer "Edge.Cuts") (width 0.1))
+  (gr_text "JLCJLCJLCJLC" (at 98.9 91.7 270) (layer "B.SilkS")
+    (effects (font (size 1 1) (thickness 0.15)) (justify mirror))
+  )
   (gr_text "4" (at 101.61044 66.4 180) (layer "F.SilkS")
     (effects (font (size 0.7 0.7) (thickness 0.12)))
