File: hardware/quad-pmod/quad-pmod.kicad_pcb (KiCad board)
At the start: 2 copper layers, 52.1 x 27.9 mm, 9 parts, among them J1 PMOD, J2 PMOD, J3 S7 Mini, J4 S7 Mini, J5 PWR, J6 PWR, J7 PMOD, J8 PMOD

Commit message: clean up routing
Routing:
- net /PORT_B1: track 14.0 -> 13.1 mm
- net /PORT_D5: track 12.3 -> 13.1 mm
- net /PORT_E2: track 11.7 -> 11.0 mm
- net /PORT_D4: track 12.3 -> 13.0 mm

Commit message: update readme following r0.1 bringup
Other:
- board text added: "JLCJLCJLC"
Changed lines of the file:
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@@
   (gr_line (start 168.148 78.994) (end 168.148 104.394) (layer "Edge.Cuts") (width 0.1))
   (gr_arc (start 166.878 104.394) (end 166.878 105.664) (angle -90) (layer "Edge.Cuts") (width 0.1))
+  (gr_text "JLCJLCJLC" (at 116.8475 91.7 270) (layer "B.SilkS")
+    (effects (font (size 1 1) (thickness 0.15)) (justify mirror))
+  )
   (gr_text "5V" (at 141.478 94.234) (layer "B.SilkS")
     (effects (font (size 1 1) (thickness 0.15)) (justify mirror))
