File: breakouts/octa-pmod-horizontal/octa-pmod.kicad_sch (KiCad schematic)
At the start: 21 parts, among them J1 PMOD, J10 PMOD, J12 PWR, J14 PWR, J15 PMOD, J16 PMOD, J2 PMOD, J3 S7 Mini, J4 S7 Mini, J5 PWR, J6 PWR, J7 PMOD, J8 PMOD, J9 PMOD, M1 M3, M2 M3, M3 M3, M4 M3

Commit message: update BOM
Parts:
- gave numbers to parts that had none: 2
Connections:
- net PORT_A0: now also J10.4 (Pin_4); no longer J10.1 (Pin_1)
- net PORT_A1: now also J10.3 (Pin_3); no longer J10.2 (Pin_2)
- net PORT_A2: now also J10.2 (Pin_2); no longer J10.3 (Pin_3)
- net PORT_A3: now also J10.1 (Pin_1); no longer J10.4 (Pin_4)
- net PORT_A4: now also J10.10 (Pin_10); no longer J10.7 (Pin_7)
- net PORT_A5: now also J10.9 (Pin_9); no longer J10.8 (Pin_8)
- net PORT_A6: now also J10.8 (Pin_8); no longer J10.9 (Pin_9)
- net PORT_A7: now also J10.7 (Pin_7); no longer J10.10 (Pin_10)
- net PORT_B0: now also J1.4 (Pin_4); no longer J1.1 (Pin_1)
- net PORT_B1: now also J1.3 (Pin_3); no longer J1.2 (Pin_2)
- net PORT_B2: now also J1.2 (Pin_2); no longer J1.3 (Pin_3)
- net PORT_B3: now also J1.1 (Pin_1); no longer J1.4 (Pin_4)
- net PORT_B4: now also J1.10 (Pin_10); no longer J1.7 (Pin_7)
- net PORT_B5: now also J1.9 (Pin_9); no longer J1.8 (Pin_8)
- net PORT_B6: now also J1.8 (Pin_8); no longer J1.9 (Pin_9)
- net PORT_B7: now also J1.7 (Pin_7); no longer J1.10 (Pin_10)
- net PORT_C0: now also J2.4 (Pin_4); no longer J2.1 (Pin_1)
- net PORT_C1: now also J2.3 (Pin_3); no longer J2.2 (Pin_2)
- net PORT_C2: now also J2.2 (Pin_2); no longer J2.3 (Pin_3)
- net PORT_C3: now also J2.1 (Pin_1); no longer J2.4 (Pin_4)
- net PORT_C4: now also J2.10 (Pin_10); no longer J2.7 (Pin_7)
- net PORT_C5: now also J2.9 (Pin_9); no longer J2.8 (Pin_8)
- net PORT_C6: now also J2.8 (Pin_8); no longer J2.9 (Pin_9)
- net PORT_C7: now also J2.7 (Pin_7); no longer J2.10 (Pin_10)
- net PORT_D0: now also J9.4 (Pin_4); no longer J9.1 (Pin_1)
- net PORT_D1: now also J9.3 (Pin_3); no longer J9.2 (Pin_2)
- net PORT_D2: now also J9.2 (Pin_2); no longer J9.3 (Pin_3)
- net PORT_D3: now also J9.1 (Pin_1); no longer J9.4 (Pin_4)
- net PORT_D4: now also J9.10 (Pin_10); no longer J9.7 (Pin_7)
- net PORT_D5: now also J9.9 (Pin_9); no longer J9.8 (Pin_8)
- net PORT_D6: now also J9.8 (Pin_8); no longer J9.9 (Pin_9)
- net PORT_D7: now also J9.7 (Pin_7); no longer J9.10 (Pin_10)
