File: hardware/0.2/ecp5-mini.kicad_sch (KiCad schematic)
At the start: 22 parts, among them J3 S7 Mini, J4 S7 Mini, U1 ECP5U_12_CABGA256, X1 DSC6101CI2A-016.0000

Commit message: almost there
Changed lines of the file:
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@@
     (company "Josh Johnson")
   )
-  (bus_alias "SD" (members "SD_DAT[0..3]" "SD_CMD" "SD_CLK" "SD_DET"))
-  (bus_alias "USB" (members "USB_D-" "USB_D+" "USB_PU"))
-  (bus_alias "HYPERRAM" (members "HR_nRST" "HR_nCS" "HR_CK_N" "HR_RWDS" "HR_DQ[0..7]" "HR_CK_P" "HR_nCK"))
   (bus_alias "LED" (members "LED_[0..7]" "LED_R" "LED_G" "LED_B"))
+  (bus_alias "HYPERRAM" (members "HR_nRST" "HR_nCS" "HR_CK_N" "HR_RWDS" "HR_DQ[0..7]" "HR_CK_P" "HR_nCK"))
+  (bus_alias "USB" (members "USB_D-" "USB_D+" "USB_PU"))
+  (bus_alias "SD" (members "SD_DAT[0..3]" "SD_CMD" "SD_CLK" "SD_DET"))
   (junction (at 60.96 58.42) (diameter 1.016) (color 0 0 0 0))
   (junction (at 62.23 176.53) (diameter 1.016) (color 0 0 0 0))
@@
   (junction (at 358.14 196.85) (diameter 1.016) (color 0 0 0 0))
   (junction (at 358.14 198.12) (diameter 1.016) (color 0 0 0 0))
-  (no_connect (at 218.44 99.06))
-  (no_connect (at 218.44 88.9))
-  (no_connect (at 138.43 250.19))
-  (no_connect (at 50.8 198.12))
-  (no_connect (at 50.8 274.32))
-  (no_connect (at 137.16 160.02))
-  (no_connect (at 50.8 101.6))
-  (no_connect (at 50.8 233.68))
-  (no_connect (at 215.9 218.44))
-  (no_connect (at 50.8 203.2))
-  (no_connect (at 138.43 262.89))
-  (no_connect (at 137.16 86.36))
-  (no_connect (at 138.43 219.71))
-  (no_connect (at 215.9 236.22))
-  (no_connect (at 50.8 238.76))
-  (no_connect (at 50.8 213.36))
-  (no_connect (at 137.16 109.22))
-  (no_connect (at 218.44 109.22))
-  (no_connect (at 137.16 157.48))
-  (no_connect (at 138.43 214.63))
   (no_connect (at 50.8 215.9))
+  (no_connect (at 137.16 88.9))
   (no_connect (at 215.9 208.28))
+  (no_connect (at 218.44 149.86))
+  (no_connect (at 50.8 269.24))
+  (no_connect (at 215.9 203.2))
+  (no_connect (at 50.8 213.36))
   (no_connect (at 50.8 236.22))
   (no_connect (at 218.44 139.7))
-  (no_connect (at 218.44 86.36))
+  (no_connect (at 137.16 86.36))
+  (no_connect (at 215.9 200.66))
+  (no_connect (at 137.16 99.06))
   (no_connect (at 138.43 273.05))
-  (no_connect (at 50.8 104.14))
-  (no_connect (at 50.8 91.44))
-  (no_connect (at 218.44 160.02))
   (no_connect (at 50.8 129.54))
-  (no_connect (at 138.43 222.25))
-  (no_connect (at 215.9 271.78))
-  (no_connect (at 50.8 210.82))
-  (no_connect (at 218.44 106.68))
-  (no_connect (at 138.43 270.51))
-  (no_connect (at 215.9 203.2))
-  (no_connect (at 215.9 220.98))
-  (no_connect (at 50.8 106.68))
+  (no_connect (at 218.44 157.48))
+  (no_connect (at 218.44 127))
+  (no_connect (at 137.16 149.86))
+  (no_connect (at 50.8 251.46))
+  (no_connect (at 218.44 99.06))
+  (no_connect (at 215.9 215.9))
+  (no_connect (at 50.8 109.22))
+  (no_connect (at 218.44 88.9))
   (no_connect (at 215.9 205.74))
+  (no_connect (at 215.9 238.76))
+  (no_connect (at 137.16 119.38))
+  (no_connect (at 218.44 109.22))
+  (no_connect (at 50.8 266.7))
+  (no_connect (at 50.8 238.76))
+  (no_connect (at 215.9 271.78))
+  (no_connect (at 137.16 121.92))
+  (no_connect (at 137.16 160.02))
+  (no_connect (at 215.9 269.24))
+  (no_connect (at 218.44 160.02))
+  (no_connect (at 50.8 259.08))
+  (no_connect (at 215.9 218.44))
   (no_connect (at 50.8 256.54))
+  (no_connect (at 215.9 266.7))
+  (no_connect (at 218.44 96.52))
+  (no_connect (at 50.8 119.38))
   (no_connect (at 137.16 116.84))
-  (no_connect (at 218.44 157.48))
-  (no_connect (at 215.9 223.52))
-  (no_connect (at 215.9 246.38))
-  (no_connect (at 138.43 252.73))
-  (no_connect (at 138.43 217.17))
-  (no_connect (at 137.16 99.06))
-  (no_connect (at 218.44 129.54))
+  (no_connect (at 138.43 242.57))
+  (no_connect (at 137.16 96.52))
+  (no_connect (at 50.8 116.84))
+  (no_connect (at 218.44 106.68))
+  (no_connect (at 50.8 198.12))
+  (no_connect (at 215.9 236.22))
   (no_connect (at 50.8 254))
-  (no_connect (at 50.8 121.92))
-  (no_connect (at 218.44 96.52))
+  (no_connect (at 137.16 109.22))
+  (no_connect (at 137.16 154.94))
+  (no_connect (at 50.8 101.6))
+  (no_connect (at 218.44 129.54))
   (no_connect (at 137.16 124.46))
-  (no_connect (at 50.8 266.7))
-  (no_connect (at 215.9 261.62))
-  (no_connect (at 215.9 215.9))
-  (no_connect (at 50.8 271.78))
-  (no_connect (at 215.9 269.24))
-  (no_connect (at 137.16 96.52))
-  (no_connect (at 137.16 119.38))
-  (no_connect (at 218.44 137.16))
-  (no_connect (at 138.43 260.35))
+  (no_connect (at 50.8 233.68))
   (no_connect (at 50.8 132.08))
-  (no_connect (at 137.16 106.68))
-  (no_connect (at 137.16 154.94))
-  (no_connect (at 218.44 127))
-  (no_connect (at 50.8 109.22))
-  (no_connect (at 50.8 116.84))
+  (no_connect (at 138.43 240.03))
+  (no_connect (at 138.43 262.89))
+  (no_connect (at 50.8 106.68))
+  (no_connect (at 50.8 203.2))
+  (no_connect (at 138.43 252.73))
+  (no_connect (at 50.8 121.92))
   (no_connect (at 50.8 127))
-  (no_connect (at 50.8 259.08))
-  (no_connect (at 215.9 200.66))
-  (no_connect (at 137.16 88.9))
-  (no_connect (at 50.8 119.38))
+  (no_connect (at 50.8 210.82))
+  (no_connect (at 138.43 217.17))
+  (no_connect (at 215.9 246.38))
+  (no_connect (at 50.8 104.14))
+  (no_connect (at 138.43 260.35))
+  (no_connect (at 215.9 220.98))
+  (no_connect (at 138.43 270.51))
   (no_connect (at 218.44 147.32))
-  (no_connect (at 137.16 149.86))
-  (no_connect (at 50.8 269.24))
-  (no_connect (at 215.9 266.7))
-  (no_connect (at 138.43 240.03))
+  (no_connect (at 138.43 222.25))
+  (no_connect (at 137.16 106.68))
+  (no_connect (at 215.9 223.52))
+  (no_connect (at 50.8 274.32))
+  (no_connect (at 138.43 219.71))
+  (no_connect (at 138.43 250.19))
+  (no_connect (at 137.16 157.48))
+  (no_connect (at 218.44 86.36))
   (no_connect (at 50.8 228.6))
-  (no_connect (at 138.43 242.57))
-  (no_connect (at 137.16 121.92))
-  (no_connect (at 218.44 149.86))
-  (no_connect (at 50.8 251.46))
-  (no_connect (at 215.9 238.76))
+  (no_connect (at 218.44 137.16))
+  (no_connect (at 215.9 261.62))
+  (no_connect (at 138.43 214.63))
+  (no_connect (at 50.8 271.78))
+  (no_connect (at 50.8 91.44))
   (bus_entry (at 62.23 81.28) (size 2.54 -2.54)
     (stroke (width 0.1524) (type solid) (color 0 0 0 0))
@@
     (stroke (width 0) (type solid) (color 0 0 0 0))
   )
-  (bus (pts (xy 64.77 77.47) (xy 64.77 91.44))
+  (bus (pts (xy 64.77 77.47) (xy 64.77 78.74))
     (stroke (width 0) (type solid) (color 0 0 0 0))
   )
@@
     (stroke (width 0) (type solid) (color 0 0 0 0))
   )
+  (bus (pts (xy 64.77 78.74) (xy 64.77 81.28))
+    (stroke (width 0) (type solid) (color 0 0 0 0))
+  )
+  (bus (pts (xy 64.77 81.28) (xy 64.77 83.82))
+    (stroke (width 0) (type solid) (color 0 0 0 0))
+  )
+  (bus (pts (xy 64.77 83.82) (xy 64.77 86.36))
+    (stroke (width 0) (type solid) (color 0 0 0 0))
+  )
+  (bus (pts (xy 64.77 86.36) (xy 64.77 91.44))
+    (stroke (width 0) (type solid) (color 0 0 0 0))
+  )
   (bus (pts (xy 64.77 91.44) (xy 64.77 93.98))
     (stroke (width 0) (type solid) (color 0 0 0 0))
@@
     (effects (font (size 2.54 2.54)) (justify right bottom))
   )
-  (text "Bank 7 (Left)" (at 121.92 184.785 180)
+  (text "Bank 6 (Left)" (at 121.92 70.485 180)
     (effects (font (size 2.54 2.54)) (justify right bottom))
   )
-  (text "Bank 6 (Left)" (at 124.46 70.485 180)
+  (text "Bank 7 (Left)" (at 121.92 184.785 180)
     (effects (font (size 2.54 2.54)) (justify right bottom))
   )
@@
     (in_bom yes) (on_board yes)
     (property "Reference" "X1" (id 0) (at 339.09 191.77 0))
-    (property "Value" "DSC6101CI2A-016.0000 " (id 1) (at 346.71 194.31 0))
+    (property "Value" "DSC6101CI2A-016.0000 " (id 1) (at 345.44 194.31 0))
     (property "Footprint" "josh-oscillators:CDFN_3.2x2.5mm_XO" (id 2) (at 347.98 186.69 0)
       (effects (font (size 2.54 2.54)) hide)
@@
     )
     (path "/d00c7eb5-4315-486e-b6f1-64546df11a37/8b2e612f-837f-449d-bfa8-23818b031dcb"
-      (reference "R1") (unit 1) (value "360K") (footprint "Resistor_SMD:R_0402_1005Metric")
+      (reference "R1") (unit 1) (value "120K") (footprint "Resistor_SMD:R_0402_1005Metric")
     )
     (path "/d00c7eb5-4315-486e-b6f1-64546df11a37/5ee8784f-ba22-4f04-a2fd-cb59772b314d"
-      (reference "R2") (unit 1) (value "82K") (footprint "Resistor_SMD:R_0402_1005Metric")
+      (reference "R2") (unit 1) (value "26K7") (footprint "Resistor_SMD:R_0402_1005Metric")
     )
     (path "/d00c7eb5-4315-486e-b6f1-64546df11a37/5cf43eb0-dbfb-4bb9-bd32-7bd945fceb1c"

Commit message: shipped 0.2
Parts:
- added FID1, FID2, FID3, FID500, FID501, FID502: Fiducial, Fiducial:Fiducial_0.5mm_Mask1mm, symbol Mechanical:Fiducial
- C1: renamed from C14; LCSC C1525 -> C327009; MPN CL05B104KO5NNNC -> CC0402KRX7R7BB103; MPN2 (none) -> CL05B104KO5NNNC; Manufacturer Samsung Electro-Mechanics -> Yageo; Manufacturer2 (none) -> Samsung Electro-Mechanics
- C502: renamed from C23; LCSC C318563 -> C326586; MPN CL05A475MO5NUNC -> CC0402KRX5R6BB475; MPN2 (none) -> CL05A475KP5NRNC; Manufacturer Samsung Electro-Mechanics -> Yageo; Manufacturer2 (none) -> Samsung Electro-Mechanics
- C503: renamed from C29; LCSC C318563 -> C326586; MPN CL05A475MO5NUNC -> CC0402KRX5R6BB475; MPN2 (none) -> CL05A475KP5NRNC; Manufacturer Samsung Electro-Mechanics -> Yageo; Manufacturer2 (none) -> Samsung Electro-Mechanics
- C504: renamed from C19; LCSC C1525 -> C327009; MPN CL05B104KO5NNNC -> CC0402KRX7R7BB103; MPN2 (none) -> CL05B104KO5NNNC; Manufacturer Samsung Electro-Mechanics -> Yageo; Manufacturer2 (none) -> Samsung Electro-Mechanics
- C505: renamed from C25; LCSC C1525 -> C327009; MPN CL05B104KO5NNNC -> CC0402KRX7R7BB103; MPN2 (none) -> CL05B104KO5NNNC; Manufacturer Samsung Electro-Mechanics -> Yageo; Manufacturer2 (none) -> Samsung Electro-Mechanics
- C510: renamed from C20; LCSC C1525 -> C327009; MPN CL05B104KO5NNNC -> CC0402KRX7R7BB103; MPN2 (none) -> CL05B104KO5NNNC; Manufacturer Samsung Electro-Mechanics -> Yageo; Manufacturer2 (none) -> Samsung Electro-Mechanics
- C511: renamed from C26; LCSC C1525 -> C327009; MPN CL05B104KO5NNNC -> CC0402KRX7R7BB103; MPN2 (none) -> CL05B104KO5NNNC; Manufacturer Samsung Electro-Mechanics -> Yageo; Manufacturer2 (none) -> Samsung Electro-Mechanics
- C512: renamed from C30; LCSC C318563 -> C326586; MPN CL05A475MO5NUNC -> CC0402KRX5R6BB475; MPN2 (none) -> CL05A475KP5NRNC; Manufacturer Samsung Electro-Mechanics -> Yageo; Manufacturer2 (none) -> Samsung Electro-Mechanics
- C514: renamed from C32; LCSC C1525 -> C327009; MPN CL05B104KO5NNNC -> CC0402KRX7R7BB103; MPN2 (none) -> CL05B104KO5NNNC; Manufacturer Samsung Electro-Mechanics -> Yageo; Manufacturer2 (none) -> Samsung Electro-Mechanics
- C520: renamed from C31; LCSC C1525 -> C327009; MPN CL05B104KO5NNNC -> CC0402KRX7R7BB103; MPN2 (none) -> CL05B104KO5NNNC; Manufacturer Samsung Electro-Mechanics -> Yageo; Manufacturer2 (none) -> Samsung Electro-Mechanics
- D10: renamed from D12; value PINK -> Pink
- D12: renamed from D1; value PINK -> Pink
- D9: renamed from D3; value PINK -> Pink
- R500: renamed from R22; LCSC C25867 -> C114451; MPN 0402WGF1501TCE -> RC0402JR-071K5L; MPN2 (none) -> 0402WGF1501TCE; Manufacturer UNI-ROYAL(Uniroyal Elec) -> Yageo; Manufacturer2 (none) -> UNI-ROYAL(Uniroyal Elec)
- R502: renamed from R5; LCSC C25867 -> C114451; MPN 0402WGF1501TCE -> RC0402JR-071K5L; MPN2 (none) -> 0402WGF1501TCE; Manufacturer UNI-ROYAL(Uniroyal Elec) -> Yageo; Manufacturer2 (none) -> UNI-ROYAL(Uniroyal Elec)
- R503: renamed from R23; LCSC C25867 -> C114451; MPN 0402WGF1501TCE -> RC0402JR-071K5L; MPN2 (none) -> 0402WGF1501TCE; Manufacturer UNI-ROYAL(Uniroyal Elec) -> Yageo; Manufacturer2 (none) -> UNI-ROYAL(Uniroyal Elec)
- U2: renamed from U1; MPN2 (none) -> LFE5U12F8BG256I; Manufacturer2 (none) -> Lattice Semiconductor; Mouser 842-LFE5U12F8BG256C -> (none)
- X1: value DSC6101CI2A-016.0000 -> 16MHz; LCSC (none) -> C387369; MPN2 (none) -> S3D16.000000B20F30T; Manufacturer2 (none) -> Shenzhen SCTF Elec; Mouser 579-101CI2A0160000 -> (none)
Other:
- moved on the sheet: J3, J4
