File: hardware/0.2/fpga-config.kicad_sch (KiCad schematic)
At the start: 30 parts, among them J2 JTAG, J5 USB_C_Receptacle_USB2.0, Q1 BSS138, SW1 PTS810, U1 ECP5U_12_CABGA256, U4 USBLC6-2P6, U6 W25Q128JVPIQ

Commit message: unrouted = 0
Changed lines of the file:
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@@
     (company "Josh Johnson")
   )
-  (bus_alias "CONFIG" (members "CFG_CLK" "CFG_IO[0..3]" "CFG_CDONE" "CFG_CS"))
+  (bus_alias "CFG" (members "CFG_CLK" "CFG_IO[0..3]" "CFG_CDONE" "CFG_CS"))
   (junction (at 27.305 74.93) (diameter 1.016) (color 0 0 0 0))
   (junction (at 46.99 35.56) (diameter 1.016) (color 0 0 0 0))
@@
   (junction (at 269.24 57.15) (diameter 1.016) (color 0 0 0 0))
   (junction (at 269.24 71.12) (diameter 1.016) (color 0 0 0 0))
+  (no_connect (at 229.87 137.16))
+  (no_connect (at 229.87 119.38))
+  (no_connect (at 229.87 142.24))
+  (no_connect (at 229.87 111.76))
+  (no_connect (at 229.87 116.84))
   (no_connect (at 229.87 121.92))
   (no_connect (at 46.355 63.5))
-  (no_connect (at 229.87 111.76))
-  (no_connect (at 229.87 116.84))
   (no_connect (at 46.355 66.04))
-  (no_connect (at 229.87 119.38))
   (no_connect (at 229.87 144.78))
-  (no_connect (at 229.87 137.16))
-  (no_connect (at 229.87 142.24))
   (bus_entry (at 114.935 49.53) (size 2.54 -2.54)
     (stroke (width 0.1524) (type solid) (color 0 0 0 0))
@@
     (effects (font (size 1.27 1.27)) (justify left bottom))
   )
-  (label "{CONFIG}" (at 215.9 45.72 270)
+  (label "{CFG}" (at 215.9 45.72 270)
     (effects (font (size 1.27 1.27)) (justify right bottom))
   )

Commit message: almost there
Other:
- note added: "IO / can be used as dfu button"
- note removed: "IO / configure to jump to bootloader"
- moved on the sheet: C13, C15, C17, C18, C6, D2, F1, J2, J5, Q1, R10, R11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

Commit message: shipped 0.2
Parts:
- C16: renamed from C6; LCSC C318563 -> C326586; MPN CL05A475MO5NUNC -> CC0402KRX5R6BB475; MPN2 (none) -> CL05A475KP5NRNC; Manufacturer Samsung Electro-Mechanics -> Yageo; Manufacturer2 (none) -> Samsung Electro-Mechanics
- C516: renamed from C17; LCSC C1525 -> C327009; MPN CL05B104KO5NNNC -> CC0402KRX7R7BB103; MPN2 (none) -> CL05B104KO5NNNC; Manufacturer Samsung Electro-Mechanics -> Yageo; Manufacturer2 (none) -> Samsung Electro-Mechanics
- C521: renamed from C15; LCSC C1525 -> C327009; MPN CL05B104KO5NNNC -> CC0402KRX7R7BB103; MPN2 (none) -> CL05B104KO5NNNC; Manufacturer Samsung Electro-Mechanics -> Yageo; Manufacturer2 (none) -> Samsung Electro-Mechanics
- C522: renamed from C18; LCSC C1525 -> C327009; MPN CL05B104KO5NNNC -> CC0402KRX7R7BB103; MPN2 (none) -> CL05B104KO5NNNC; Manufacturer Samsung Electro-Mechanics -> Yageo; Manufacturer2 (none) -> Samsung Electro-Mechanics
- C523: renamed from C13; LCSC C1525 -> C327009; MPN CL05B104KO5NNNC -> CC0402KRX7R7BB103; MPN2 (none) -> CL05B104KO5NNNC; Manufacturer Samsung Electro-Mechanics -> Yageo; Manufacturer2 (none) -> Samsung Electro-Mechanics
- D11: renamed from D2; value PINK -> Pink
- F1: MPN2 (none) -> JK-SMD0603-100L; Manufacturer2 (none) -> Jinrui Electronic Materials Co.
- J5: value USB_C_Receptacle_USB2.0 -> USB_Type_C_2.0; MPN TYPE-C-31-M-12 -> USB4105-GF-A; MPN2 (none) -> TYPE-C-31-M-12; Manufacturer Korean Hroparts Elec -> GCT; Manufacturer2 (none) -> Korean Hroparts Elec; Notes Digikey: USB4105-GF-A -> (none)
- Q500: renamed from Q1; MPN2 (none) -> BSS138W-7-F; Manufacturer2 (none) -> Diodes Incorporated
- R501: renamed from R21; LCSC C25867 -> C114451; MPN 0402WGF1501TCE -> RC0402JR-071K5L; MPN2 (none) -> 0402WGF1501TCE; Manufacturer UNI-ROYAL(Uniroyal Elec) -> Yageo; Manufacturer2 (none) -> UNI-ROYAL(Uniroyal Elec)
- R504: renamed from R7; LCSC C25905 -> C105873; MPN 0402WGF5101TCE -> RC0402JR-075K1L; MPN2 (none) -> 0402WGF5101TCE; Manufacturer UNI-ROYAL(Uniroyal Elec) -> Yageo; Manufacturer2 (none) -> UNI-ROYAL(Uniroyal Elec)
- R505: renamed from R6; LCSC C25905 -> C105873; MPN 0402WGF5101TCE -> RC0402JR-075K1L; MPN2 (none) -> 0402WGF5101TCE; Manufacturer UNI-ROYAL(Uniroyal Elec) -> Yageo; Manufacturer2 (none) -> UNI-ROYAL(Uniroyal Elec)
- R506: renamed from R10; LCSC C25152 -> C93929; MPN 0402WGJ0220TCE -> RC0402JR-0722RL; MPN2 (none) -> 0402WGJ0220TCE; Manufacturer UNI-ROYAL(Uniroyal Elec) -> Yageo; Manufacturer2 (none) -> UNI-ROYAL(Uniroyal Elec)
- R507: renamed from R9; LCSC C25152 -> C93929; MPN 0402WGJ0220TCE -> RC0402JR-0722RL; MPN2 (none) -> 0402WGJ0220TCE; Manufacturer UNI-ROYAL(Uniroyal Elec) -> Yageo; Manufacturer2 (none) -> UNI-ROYAL(Uniroyal Elec)
- R508: renamed from R11; LCSC C25867 -> C114451; MPN 0402WGF1501TCE -> RC0402JR-071K5L; MPN2 (none) -> 0402WGF1501TCE; Manufacturer UNI-ROYAL(Uniroyal Elec) -> Yageo; Manufacturer2 (none) -> UNI-ROYAL(Uniroyal Elec)
- R509: renamed from R20; LCSC C25152 -> C93929; MPN 0402WGJ0220TCE -> RC0402JR-0722RL; MPN2 (none) -> 0402WGJ0220TCE; Manufacturer UNI-ROYAL(Uniroyal Elec) -> Yageo; Manufacturer2 (none) -> UNI-ROYAL(Uniroyal Elec)
- R511: renamed from R19; LCSC C25905 -> C105873; MPN 0402WGF5101TCE -> RC0402JR-075K1L; MPN2 (none) -> 0402WGF5101TCE; Manufacturer UNI-ROYAL(Uniroyal Elec) -> Yageo; Manufacturer2 (none) -> UNI-ROYAL(Uniroyal Elec)
- R512: renamed from R29; LCSC C25531 -> C60489; MPN 0402WGJ0103TCE -> RC0402JR-0710KL; MPN2 (none) -> 0402WGJ0103TCE; Manufacturer UNI-ROYAL(Uniroyal Elec) -> Yageo; Manufacturer2 (none) -> UNI-ROYAL(Uniroyal Elec)
- R514: renamed from R24; LCSC C25531 -> C60489; MPN 0402WGJ0103TCE -> RC0402JR-0710KL; MPN2 (none) -> 0402WGJ0103TCE; Manufacturer UNI-ROYAL(Uniroyal Elec) -> Yageo; Manufacturer2 (none) -> UNI-ROYAL(Uniroyal Elec)
- R516: renamed from R12; LCSC C25905 -> C105873; MPN 0402WGF5101TCE -> RC0402JR-075K1L; MPN2 (none) -> 0402WGF5101TCE; Manufacturer UNI-ROYAL(Uniroyal Elec) -> Yageo; Manufacturer2 (none) -> UNI-ROYAL(Uniroyal Elec)
- R517: renamed from R8; LCSC C25531 -> C60489; MPN 0402WGJ0103TCE -> RC0402JR-0710KL; MPN2 (none) -> 0402WGJ0103TCE; Manufacturer UNI-ROYAL(Uniroyal Elec) -> Yageo; Manufacturer2 (none) -> UNI-ROYAL(Uniroyal Elec)
- R518: renamed from R26; LCSC C25531 -> C60489; MPN 0402WGJ0103TCE -> RC0402JR-0710KL; MPN2 (none) -> 0402WGJ0103TCE; Manufacturer UNI-ROYAL(Uniroyal Elec) -> Yageo; Manufacturer2 (none) -> UNI-ROYAL(Uniroyal Elec)
- R519: renamed from R27; LCSC C25531 -> C60489; MPN 0402WGJ0103TCE -> RC0402JR-0710KL; MPN2 (none) -> 0402WGJ0103TCE; Manufacturer UNI-ROYAL(Uniroyal Elec) -> Yageo; Manufacturer2 (none) -> UNI-ROYAL(Uniroyal Elec)
- SW1: MPN2 (none) -> SKRPACE010; Manufacturer2 (none) -> Alps
- U1: renamed from U6; Mouser 454-W25Q128JVPIQ -> (none)
- U2: renamed from U1; MPN2 (none) -> LFE5U12F8BG256I; Manufacturer2 (none) -> Lattice Semiconductor; Mouser 842-LFE5U12F8BG256C -> (none)
- U6: renamed from U4; Mouser 511-USBLC6-2P6 -> (none)
- renumbered TP1 to TP500, TP2 to TP501
Other:
- note added: "Button can be configured for DFU"
- note removed: "IO / can be used as dfu button"

Commit message: checking for the final time
Parts:
- R504, R505, R511, R516: MPN RC0402JR-075K1L -> RC0402JR-075K1L
- R512, R514, R517, R518, R519: MPN RC0402JR-0710KL -> RC0402JR-0710KL
Changed lines of the file:
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@@
   (no_connect (at 208.28 151.13))
   (no_connect (at 208.28 148.59))
+  (no_connect (at 52.07 82.55))
+  (no_connect (at 208.28 125.73))
+  (no_connect (at 52.07 80.01))
+  (no_connect (at 208.28 118.11))
   (no_connect (at 208.28 123.19))
+  (no_connect (at 208.28 143.51))
   (no_connect (at 208.28 128.27))
-  (no_connect (at 208.28 143.51))
-  (no_connect (at 52.07 80.01))
-  (no_connect (at 52.07 82.55))
-  (no_connect (at 208.28 118.11))
-  (no_connect (at 208.28 125.73))
   (bus_entry (at 120.65 66.04) (size 2.54 -2.54)
     (stroke (width 0.1524) (type solid) (color 0 0 0 0))
@@
       (effects (font (size 1.27 1.27)) hide)
     )
-    (property "MPN" "RC0402JR-075K1L" (id 5) (at 57.15 57.15 0)
+    (property "MPN" "RC0402JR-075K1L\n" (id 5) (at 57.15 57.15 0)
       (effects (font (size 1.27 1.27)) hide)
     )
@@
       (effects (font (size 1.27 1.27)) hide)
     )
-    (property "MPN" "RC0402JR-075K1L" (id 5) (at 57.15 59.69 0)
+    (property "MPN" "RC0402JR-075K1L\n" (id 5) (at 57.15 59.69 0)
       (effects (font (size 1.27 1.27)) hide)
     )
@@
       (effects (font (size 1.27 1.27)) hide)
     )
-    (property "MPN" "RC0402JR-0710KL" (id 5) (at 66.04 147.32 0)
+    (property "MPN" "RC0402JR-0710KL\n" (id 5) (at 66.04 147.32 0)
       (effects (font (size 1.27 1.27)) hide)
     )
@@
       (effects (font (size 1.27 1.27)) (justify left top))
     )
-    (property "MPN" "RC0402JR-075K1L" (id 5) (at 146.05 148.59 0)
+    (property "MPN" "RC0402JR-075K1L\n" (id 5) (at 146.05 148.59 0)
       (effects (font (size 1.27 1.27)) hide)
     )
@@
       (effects (font (size 1.27 1.27)) (justify left top))
     )
-    (property "MPN" "RC0402JR-075K1L" (id 5) (at 168.91 148.59 0)
+    (property "MPN" "RC0402JR-075K1L\n" (id 5) (at 168.91 148.59 0)
       (effects (font (size 1.27 1.27)) hide)
     )
@@
       (effects (font (size 1.27 1.27)) hide)
     )
-    (property "MPN" "RC0402JR-0710KL" (id 5) (at 200.66 53.34 0)
+    (property "MPN" "RC0402JR-0710KL\n" (id 5) (at 200.66 53.34 0)
       (effects (font (size 1.27 1.27)) hide)
     )
@@
       (effects (font (size 1.27 1.27)) hide)
     )
-    (property "MPN" "RC0402JR-0710KL" (id 5) (at 208.28 53.34 0)
+    (property "MPN" "RC0402JR-0710KL\n" (id 5) (at 208.28 53.34 0)
       (effects (font (size 1.27 1.27)) hide)
     )
@@
       (effects (font (size 1.27 1.27)) hide)
     )
-    (property "MPN" "RC0402JR-0710KL" (id 5) (at 215.9 53.34 0)
+    (property "MPN" "RC0402JR-0710KL\n" (id 5) (at 215.9 53.34 0)
       (effects (font (size 1.27 1.27)) hide)
     )
@@
       (effects (font (size 1.27 1.27)) hide)
     )
-    (property "MPN" "RC0402JR-0710KL" (id 5) (at 224.79 53.34 0)
-      (effects (font (size 1.27 1.27)) hide)
-    )
+    (property "MPN" "RC0402JR-0710KL\n" (id 5) (at 224.79 53.34 0)
+      (effects (font (size 1.27 1.27)) hide)
+    )
