File: hardware/0.2/power.kicad_sch (KiCad schematic)
At the start: 32 parts, among them U1 ECP5U_12_CABGA256, U2 TLV75525PDQNR, U3 TLV75518PDQNR, U5 TLV62569DRLR, U8 TLV62569DRLR

Commit message: almost there
Parts:
- R1: value 360K -> 120K; LCSC C45956 -> C25750; MPN 0402WGF3603TCE -> 0402WGF1203TCE
- R2: value 82K -> 26K7; LCSC C4142 -> C138023; MPN 0402WGF8202TCE -> RC0402FR-0726K7L; Manufacturer UNI-ROYAL(Uniroyal Elec) -> YAGEO
Other:
- note added: "V_{out} = 0.6V * (1 + R1/R2) 1v1 = 0.6 * (1 + 100k/120k) 1v1 @ 1A"
- note added: "V_{out} = 0.6V * (1 + R1/R2) 3v3 = 0.6 * (1 + 120k/26.7k) 3v3 @ 1A"
- note removed: "V_{out} = 0.6V * (1 + R1/R2) 1v11 = 0.6 * (1 + 84k5/100k) 1v1 @ 1A"
- note removed: "V_{out} = 0.6V * (1 + R1/R2) 3v28 = 0.6 * (1 + 210k/47k) 3v3 @ 1A"
- moved on the sheet: C24, C4, U2, U3

Commit message: shipped 0.2
Parts:
- C10: renamed from C27; LCSC C92487 -> C109453; MPN CL10A106MO8NQNC -> CC0603MRX5R6BB106; MPN2 (none) -> CL10A106KP8NNNC; Manufacturer Samsung Electro-Mechanics -> Yageo; Manufacturer2 (none) -> Samsung Electro-Mechanics
- C11: renamed from C10; LCSC C92487 -> C109453; MPN CL10A106MO8NQNC -> CC0603MRX5R6BB106; MPN2 (none) -> CL10A106KP8NNNC; Manufacturer Samsung Electro-Mechanics -> Yageo; Manufacturer2 (none) -> Samsung Electro-Mechanics
- C13: renamed from C9; LCSC C86292 -> C327291; MPN CL05C6R8DB5NNNC -> CC0402KRX7R9BB682; MPN2 (none) -> CL05B682KA5NNNC; Manufacturer Samsung Electro-Mechanics -> Yageo; Manufacturer2 (none) -> Samsung Electro-Mechanics
- C14: renamed from C8; LCSC C86292 -> C327291; MPN CL05C6R8DB5NNNC -> CC0402KRX7R9BB682; MPN2 (none) -> CL05B682KA5NNNC; Manufacturer Samsung Electro-Mechanics -> Yageo; Manufacturer2 (none) -> Samsung Electro-Mechanics
- C17: renamed from C1; LCSC C318563 -> C326586; MPN CL05A475MO5NUNC -> CC0402KRX5R6BB475; MPN2 (none) -> CL05A475KP5NRNC; Manufacturer Samsung Electro-Mechanics -> Yageo; Manufacturer2 (none) -> Samsung Electro-Mechanics
- C18: renamed from C2; LCSC C318563 -> C326586; MPN CL05A475MO5NUNC -> CC0402KRX5R6BB475; MPN2 (none) -> CL05A475KP5NRNC; Manufacturer Samsung Electro-Mechanics -> Yageo; Manufacturer2 (none) -> Samsung Electro-Mechanics
- C2: renamed from C4; LCSC C318563 -> C326586; MPN CL05A475MO5NUNC -> CC0402KRX5R6BB475; MPN2 (none) -> CL05A475KP5NRNC; Manufacturer Samsung Electro-Mechanics -> Yageo; Manufacturer2 (none) -> Samsung Electro-Mechanics
- C3: LCSC C318563 -> C326586; MPN CL05A475MO5NUNC -> CC0402KRX5R6BB475; MPN2 (none) -> CL05A475KP5NRNC; Manufacturer Samsung Electro-Mechanics -> Yageo; Manufacturer2 (none) -> Samsung Electro-Mechanics
- C506: renamed from C38; LCSC C1525 -> C327009; MPN CL05B104KO5NNNC -> CC0402KRX7R7BB103; MPN2 (none) -> CL05B104KO5NNNC; Manufacturer Samsung Electro-Mechanics -> Yageo; Manufacturer2 (none) -> Samsung Electro-Mechanics
- C507: renamed from C21; LCSC C318563 -> C326586; MPN CL05A475MO5NUNC -> CC0402KRX5R6BB475; MPN2 (none) -> CL05A475KP5NRNC; Manufacturer Samsung Electro-Mechanics -> Yageo; Manufacturer2 (none) -> Samsung Electro-Mechanics
- C508: renamed from C37; LCSC C1525 -> C327009; MPN CL05B104KO5NNNC -> CC0402KRX7R7BB103; MPN2 (none) -> CL05B104KO5NNNC; Manufacturer Samsung Electro-Mechanics -> Yageo; Manufacturer2 (none) -> Samsung Electro-Mechanics
- C509: renamed from C39; LCSC C1525 -> C327009; MPN CL05B104KO5NNNC -> CC0402KRX7R7BB103; MPN2 (none) -> CL05B104KO5NNNC; Manufacturer Samsung Electro-Mechanics -> Yageo; Manufacturer2 (none) -> Samsung Electro-Mechanics
- C513: renamed from C41; LCSC C1525 -> C327009; MPN CL05B104KO5NNNC -> CC0402KRX7R7BB103; MPN2 (none) -> CL05B104KO5NNNC; Manufacturer Samsung Electro-Mechanics -> Yageo; Manufacturer2 (none) -> Samsung Electro-Mechanics
- C515: renamed from C42; LCSC C1525 -> C327009; MPN CL05B104KO5NNNC -> CC0402KRX7R7BB103; MPN2 (none) -> CL05B104KO5NNNC; Manufacturer Samsung Electro-Mechanics -> Yageo; Manufacturer2 (none) -> Samsung Electro-Mechanics
- C517: renamed from C22; LCSC C318563 -> C326586; MPN CL05A475MO5NUNC -> CC0402KRX5R6BB475; MPN2 (none) -> CL05A475KP5NRNC; Manufacturer Samsung Electro-Mechanics -> Yageo; Manufacturer2 (none) -> Samsung Electro-Mechanics
- C518: renamed from C43; LCSC C1525 -> C327009; MPN CL05B104KO5NNNC -> CC0402KRX7R7BB103; MPN2 (none) -> CL05B104KO5NNNC; Manufacturer Samsung Electro-Mechanics -> Yageo; Manufacturer2 (none) -> Samsung Electro-Mechanics
- C519: renamed from C40; LCSC C1525 -> C327009; MPN CL05B104KO5NNNC -> CC0402KRX7R7BB103; MPN2 (none) -> CL05B104KO5NNNC; Manufacturer Samsung Electro-Mechanics -> Yageo; Manufacturer2 (none) -> Samsung Electro-Mechanics
- C6: renamed from C5; LCSC C92487 -> C109453; MPN CL10A106MO8NQNC -> CC0603MRX5R6BB106; MPN2 (none) -> CL10A106KP8NNNC; Manufacturer Samsung Electro-Mechanics -> Yageo; Manufacturer2 (none) -> Samsung Electro-Mechanics
- C7: LCSC C92487 -> C109453; MPN CL10A106MO8NQNC -> CC0603MRX5R6BB106; MPN2 (none) -> CL10A106KP8NNNC; Manufacturer Samsung Electro-Mechanics -> Yageo; Manufacturer2 (none) -> Samsung Electro-Mechanics
- C8: renamed from C16; LCSC C318563 -> C326586; MPN CL05A475MO5NUNC -> CC0402KRX5R6BB475; MPN2 (none) -> CL05A475KP5NRNC; Manufacturer Samsung Electro-Mechanics -> Yageo; Manufacturer2 (none) -> Samsung Electro-Mechanics
- C9: renamed from C24; LCSC C318563 -> C326586; MPN CL05A475MO5NUNC -> CC0402KRX5R6BB475; MPN2 (none) -> CL05A475KP5NRNC; Manufacturer Samsung Electro-Mechanics -> Yageo; Manufacturer2 (none) -> Samsung Electro-Mechanics
- L1, L2: MPN SLM20122R2MIT -> LQM21PN2R2NGCD; MPN2 (none) -> SLM20122R2MIT; Manufacturer Sunltech Tech -> Murata Electronics; Manufacturer2 (none) -> Sunltech Tech
- R1, R4: LCSC C25750 -> C93945; MPN 0402WGF1203TCE -> RC0402FR-07120KL; MPN2 (none) -> 0402WGF1203TCE; Manufacturer UNI-ROYAL(Uniroyal Elec) -> Yageo; Manufacturer2 (none) -> UNI-ROYAL(Uniroyal Elec); Tolerance 1% -> (none)
- R2: renamed from R3; LCSC C25741 -> C60491; MPN 0402WGF1003TCE -> RC0402FR-07100KL; MPN2 (none) -> 0402WGF1003TCE; Manufacturer UNI-ROYAL(Uniroyal Elec) -> Yageo; Manufacturer2 (none) -> UNI-ROYAL(Uniroyal Elec); Tolerance 1% -> (none)
- R3: renamed from R2; MPN2 (none) -> ERJ-2RKF2672X; Manufacturer YAGEO -> Yageo; Manufacturer2 (none) -> Panasonic; Tolerance 1% -> (none)
- U2: renamed from U1; MPN2 (none) -> LFE5U12F8BG256I; Manufacturer2 (none) -> Lattice Semiconductor; Mouser 842-LFE5U12F8BG256C -> (none)
- U4: renamed from U2; LCSC (none) -> C603508; MPN (none) -> TLV75525PDQNR; MPN2 (none) -> NCP115CMX250TCG; Manufacturer (none) -> Texas Instruments; Manufacturer2 (none) -> ON Semiconductor
- U5: renamed from U3; LCSC (none) -> C603507; MPN (none) -> TLV75518PDQNR; MPN2 (none) -> NCP115CMX180TCG; Manufacturer (none) -> Texas Instruments; Manufacturer2 (none) -> ON Semiconductor
- U7: renamed from U5; Mouser 595-TLV62569DRLR -> (none)
- U8: Mouser 595-TLV62569DRLR -> (none)

Commit message: bom fix
Parts:
- C506, C508, C509, C513, C515, C518, C519: MPN CC0402KRX7R7BB103 -> CC0402KRX7R7BB104
Changed lines of the file:
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@@
       (effects (font (size 1.27 1.27)) hide)
     )
-    (property "MPN" "CC0402KRX7R7BB103" (id 5) (at 182.88 81.28 0)
+    (property "MPN" "CC0402KRX7R7BB104" (id 5) (at 182.88 81.28 0)
       (effects (font (size 1.27 1.27)) hide)
     )
@@
       (effects (font (size 1.27 1.27)) hide)
     )
-    (property "MPN" "CC0402KRX7R7BB103" (id 5) (at 182.88 107.95 0)
+    (property "MPN" "CC0402KRX7R7BB104" (id 5) (at 182.88 107.95 0)
       (effects (font (size 1.27 1.27)) hide)
     )
@@
       (effects (font (size 1.27 1.27)) hide)
     )
-    (property "MPN" "CC0402KRX7R7BB103" (id 5) (at 193.04 81.28 0)
+    (property "MPN" "CC0402KRX7R7BB104" (id 5) (at 193.04 81.28 0)
       (effects (font (size 1.27 1.27)) hide)
     )
@@
       (effects (font (size 1.27 1.27)) hide)
     )
-    (property "MPN" "CC0402KRX7R7BB103" (id 5) (at 193.04 107.95 0)
+    (property "MPN" "CC0402KRX7R7BB104" (id 5) (at 193.04 107.95 0)
       (effects (font (size 1.27 1.27)) hide)
     )
@@
       (effects (font (size 1.27 1.27)) hide)
     )
-    (property "MPN" "CC0402KRX7R7BB103" (id 5) (at 203.2 81.28 0)
+    (property "MPN" "CC0402KRX7R7BB104" (id 5) (at 203.2 81.28 0)
       (effects (font (size 1.27 1.27)) hide)
     )
@@
       (effects (font (size 1.27 1.27)) hide)
     )
-    (property "MPN" "CC0402KRX7R7BB103" (id 5) (at 213.36 81.28 0)
+    (property "MPN" "CC0402KRX7R7BB104" (id 5) (at 213.36 81.28 0)
       (effects (font (size 1.27 1.27)) hide)
     )
@@
       (effects (font (size 1.27 1.27)) hide)
     )
-    (property "MPN" "CC0402KRX7R7BB103" (id 5) (at 223.52 81.28 0)
+    (property "MPN" "CC0402KRX7R7BB104" (id 5) (at 223.52 81.28 0)
       (effects (font (size 1.27 1.27)) hide)
     )

Commit message: nightly version bump
Parts:
- C10, C11, C6, C7: MPN2 CL10A106KP8NNNC -> (none)
- C13, C14: Manufacturer2 Samsung Electro-Mechanics -> (none)
- C17, C18, C2, C3, C507, C517, C8, C9: MPN2 CL05A475KP5NRNC -> (none)
- C506, C508, C509, C513, C515, C518, C519: MPN2 CL05B104KO5NNNC -> (none)
- L1, L2: MPN2 SLM20122R2MIT -> (none); Manufacturer Murata Electronics -> (none)
- R1, R4: LCSC C93945 -> (none)
- R2: LCSC C60491 -> (none)
- R3: LCSC C138023 -> (none)
